File: hardware/device.kicad_pcb (KiCad board)
At the start: 4 copper layers, 100 x 40 mm, 144 parts, among them J10 Conn_Coaxial, J3.3V1 Conn_01x02, J3.3V2 Conn_01x02, J5V1 Conn_01x02, J5V2 Conn_01x02, Q1 AO3400A, Q10 AO3401A, Q11 AO3400A, Q12 AO3401A, Q2 AO3400A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

Commit message: fix(hardware): fix 5V divider resistors
oops, i forgot some parentheses when calculating them initially
Parts:
- R19: value 1.8kΩ -> 10kΩ
- R22: value 100kΩ -> NC
Changed lines of the file:
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@@
         (effects (font (size 1 1) (thickness 0.15)))
     )
-    (fp_text value "1.8kΩ" (at 0 1.43 90) (layer "F.Fab") hide
+    (fp_text value "10kΩ" (at 0 1.43 90) (layer "F.Fab") hide
         (effects (font (size 1 1) (thickness 0.15)))
     )
@@
     (property "Sheetfile" "device.kicad_sch")
     (property "Sheetname" "")
+    (property "dnp" "")
     (property "ki_description" "Resistor")
     (property "ki_keywords" "R res resistor")
@@
         (effects (font (size 1 1) (thickness 0.15)))
     )
-    (fp_text value "100kΩ" (at 0 1.43) (layer "F.Fab") hide
-        (effects (font (size 1 1) (thickness 0.15)))
-    )
+    (fp_text value "NC" (at 0 1.43) (layer "F.Fab") hide
+        (effects (font (size 1 1) (thickness 0.15)))
+    )
