File: hardware/device.kicad_sch (KiCad schematic)
At the start: 127 parts, among them J10 Conn_Coaxial, J3.3V1 Conn_01x02, J3.3V2 Conn_01x02, J5V1 Conn_01x02, J5V2 Conn_01x02, Q1 AO3400A, Q10 AO3401A, Q11 AO3400A, Q12 AO3401A, Q2 AO3400A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

Commit message: fix(hardware): fix 5V divider resistors
oops, i forgot some parentheses when calculating them initially
Parts:
- R19: value 1.8kΩ -> 10kΩ
- R22: value 100kΩ -> NC; now not fitted
Changed lines of the file:
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@@
       (effects (font (size 1.27 1.27)))
     )
-    (property "Value" "1.8kΩ" (at 110.49 41.91 90)
+    (property "Value" "10kΩ" (at 110.49 41.91 90)
       (effects (font (size 1.27 1.27)))
     )
@@
   )
   (symbol (lib_id "Device:R") (at 111.76 31.75 0) (unit 1)
-    (in_bom yes) (on_board yes) (dnp no)
+    (in_bom yes) (on_board yes) (dnp yes)
     (property "Reference" "R22" (at 109.22 31.75 90)
       (effects (font (size 1.27 1.27)))
     )
-    (property "Value" "100kΩ" (at 114.3 31.75 90)
+    (property "Value" "NC" (at 114.3 31.75 90)
       (effects (font (size 1.27 1.27)))
     )
